Commit message: fix duplicate parent joint for frame_link

File: cenic_bench/models/trossen_stationary_ai/stationary_ai.urdf (robot description, URDF)
Before this commit: robot stationary_ai, 70 links, 70 joints
Joints:
- joint world_joint: child frame_link -> tabletop_link

Commit message: replace gripper mimic joints with independent actuators

File: cenic_bench/models/trossen_stationary_ai/stationary_ai.urdf (robot description, URDF)
Before this commit: robot stationary_ai, 70 links, 70 joints
Joints:
- joint follower_left_right_carriage_joint: mimic joint=follower_left_left_carriage_joint -> (none)
- joint follower_right_right_carriage_joint: mimic joint=follower_right_left_carriage_joint -> (none)

Commit message: Revert "replace gripper mimic joints with independent actuators"
This reverts commit bc61bd7a2a506ac9946332a561dde57026570dcd.

File: cenic_bench/models/trossen_stationary_ai/stationary_ai.urdf (robot description, URDF)
Before this commit: robot stationary_ai, 70 links, 70 joints
Joints:
- joint follower_left_right_carriage_joint: mimic (none) -> joint=follower_left_left_carriage_joint
- joint follower_right_right_carriage_joint: mimic (none) -> joint=follower_right_left_carriage_joint
